Commit message: silla de ruedas en urdf sin exito, los controladores no funcionan y tampoco meshes

File: model/wheelchair_with_lidar/wheelchair_urdf/wheelchair.urdf (robot description, URDF)
Before this commit: robot wheelchai_with_lidar, 6 links, 5 joints
Links:
- link Mainbody: geometry collision mesh filename=model://wheelchair/wheelchair_urdf/meshes/Wheelchair.stl scale=1 1 1; visual mesh filename=model://wheelchair/wheelchair_urdf/meshes/Wheelchair.stl scale=1 1 1
